File: pinkytyl_v2.kicad_pcb (KiCad board)
At the start: 2 copper layers, 132 x 105.9 mm, 58 parts, among them J1 50-00174, J2 Conn_01x02, J3 USB_B_Mini, J5 Conn_02x05_Odd_Even, K0 KEYSW, K10 KEYSW, K11 KEYSW, K12 KEYSW, K13 KEYSW, K14 KEYSW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

Commit message: Routing complete, time for review
Parts:
- moved C2 3.25 mm to (180.7, 114.1), turned to 0 degrees
- moved C4 2.04 mm to (170.0, 101.5), turned to 45 degrees
- moved C5 1.74 mm to (173.9, 101.8), turned to 135 degrees
- moved C7 1.19 mm to (179.0, 110.4), turned to 0 degrees
- moved R1 1.07 mm to (178.1, 111.9)
- moved R3 0.39 mm to (175.6, 105.9)
- moved R2 0.38 mm to (177.1, 113.0)
- turned Y1 to 135 degrees
Routing:
- net VCC: track 118.9 -> 234.0 mm, vias 4 -> 15
- net serial: track 0.00 -> 75.0 mm, vias 0 -> 2
- net GND: track 1.59 -> 59.1 mm, vias 0 -> 4
- net reset: track 0.00 -> 26.5 mm, vias 0 -> 1
- net MOSI: track 167.5 -> 193.0 mm, vias 2 -> 4
- net MISO: track 158.4 -> 169.7 mm
- net Net-(C5-Pad1): track 0.00 -> 6.89 mm
- net Net-(C4-Pad1): track 0.00 -> 6.79 mm
- net c3: track 150.0 -> 156.3 mm
- net r0: track 166.5 -> 172.1 mm
- net Net-(C7-Pad1): track 0.00 -> 4.43 mm
- net Net-(R1-Pad1): track 0.00 -> 2.69 mm
- net r2: track 142.1 -> 144.3 mm
- net Net-(R2-Pad1): track 0.00 -> 1.77 mm
- net c0: track 154.5 -> 156.3 mm
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- added copper zone on B.Cu, net GND
- added copper zone on F.Cu, net GND

Commit message: Adds mounting holes
Parts:
- added H1: MountingHole_Pad, MountingHole:MountingHole_2.2mm_M2_Pad, F.Cu at (89.4, 112.1)
- added H2: MountingHole_Pad, MountingHole:MountingHole_2.2mm_M2_Pad, F.Cu at (107.6, 73.9)
- added H3: MountingHole_Pad, MountingHole:MountingHole_2.2mm_M2_Pad, F.Cu at (146.5, 65.2)
- added H4: MountingHole_Pad, MountingHole:MountingHole_2.2mm_M2_Pad, F.Cu at (182.4, 135.6)
Changed lines of the file:
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@@
     (tracks 592)
     (zones 0)
-    (modules 58)
+    (modules 62)
     (nets 64)
   )
@@
     (add_net serial)
   )
+  (module MountingHole:MountingHole_2.2mm_M2_Pad (layer F.Cu)
+    (at 182.44 135.63)
+    (descr "Mounting Hole 2.2mm, M2")
+    (tags "mounting hole 2.2mm m2")
+    (attr virtual)
+    (fp_text reference H4 (at 0 -3.2) (layer F.SilkS)
+      (effects (font (size 1 1) (thickness 0.15)))
+    )
+    (fp_text value MountingHole_Pad (at 0 3.2) (layer F.Fab)
+      (effects (font (size 1 1) (thickness 0.15)))
+    )
+    (fp_text user %R (at 0.3 0) (layer F.Fab)
+      (effects (font (size 1 1) (thickness 0.15)))
+    )
+    (fp_circle (center 0 0) (end 2.2 0) (layer Cmts.User) (width 0.15))
+    (fp_circle (center 0 0) (end 2.45 0) (layer F.CrtYd) (width 0.05))
+    (pad 1 thru_hole circle (at 0 0) (size 4.4 4.4) (drill 2.2) (layers *.Cu *.Mask)
+      (net 2 GND))
+  )
+  (module MountingHole:MountingHole_2.2mm_M2_Pad (layer F.Cu)
+    (at 146.46 65.23)
+    (descr "Mounting Hole 2.2mm, M2")
+    (tags "mounting hole 2.2mm m2")
+    (attr virtual)
+    (fp_text reference H3 (at 0 -3.2) (layer F.SilkS)
+      (effects (font (size 1 1) (thickness 0.15)))
+    )
+    (fp_text value MountingHole_Pad (at 0 3.2) (layer F.Fab)
+      (effects (font (size 1 1) (thickness 0.15)))
+    )
+    (fp_text user %R (at 0.3 0) (layer F.Fab)
+      (effects (font (size 1 1) (thickness 0.15)))
+    )
+    (fp_circle (center 0 0) (end 2.2 0) (layer Cmts.User) (width 0.15))
+    (fp_circle (center 0 0) (end 2.45 0) (layer F.CrtYd) (width 0.05))
+    (pad 1 thru_hole circle (at 0 0) (size 4.4 4.4) (drill 2.2) (layers *.Cu *.Mask)
+      (net 2 GND))
+  )
+  (module MountingHole:MountingHole_2.2mm_M2_Pad (layer F.Cu)
+    (at 107.59 73.91)
+    (descr "Mounting Hole 2.2mm, M2")
+    (tags "mounting hole 2.2mm m2")
+    (attr virtual)
+    (fp_text reference H2 (at 0 -3.2) (layer F.SilkS)
+      (effects (font (size 1 1) (thickness 0.15)))
+    )
+    (fp_text value MountingHole_Pad (at 0 3.2) (layer F.Fab)
+      (effects (font (size 1 1) (thickness 0.15)))
+    )
+    (fp_text user %R (at 0.3 0) (layer F.Fab)
+      (effects (font (size 1 1) (thickness 0.15)))
+    )
+    (fp_circle (center 0 0) (end 2.2 0) (layer Cmts.User) (width 0.15))
+    (fp_circle (center 0 0) (end 2.45 0) (layer F.CrtYd) (width 0.05))
+    (pad 1 thru_hole circle (at 0 0) (size 4.4 4.4) (drill 2.2) (layers *.Cu *.Mask)
+      (net 2 GND))
+  )
+  (module MountingHole:MountingHole_2.2mm_M2_Pad (layer F.Cu)
+    (at 89.37 112.08)
+    (descr "Mounting Hole 2.2mm, M2")
+    (tags "mounting hole 2.2mm m2")
+    (attr virtual)
+    (fp_text reference H1 (at 0 -3.2) (layer F.SilkS)
+      (effects (font (size 1 1) (thickness 0.15)))
+    )
+    (fp_text value MountingHole_Pad (at 0 3.2) (layer F.Fab)
+      (effects (font (size 1 1) (thickness 0.15)))
+    )
+    (fp_text user %R (at 0.3 0) (layer F.Fab)
+      (effects (font (size 1 1) (thickness 0.15)))
+    )
+    (fp_circle (center 0 0) (end 2.2 0) (layer Cmts.User) (width 0.15))
+    (fp_circle (center 0 0) (end 2.45 0) (layer F.CrtYd) (width 0.05))
+    (pad 1 thru_hole circle (at 0 0) (size 4.4 4.4) (drill 2.2) (layers *.Cu *.Mask)
+      (net 2 GND))
+  )
   (module misc:54-00174 (layer F.Cu)

Commit message: Rough layout, might be ready for order
Parts:
- U1: value ATmega32U4-MU -> ATmega32U4-AU; footprint Package_DFN_QFN:QFN-44-1EP_7x7mm_P0.5mm_EP5.2x5.2mm -> Package_QFP:TQFP-44_10x10mm_P0.8mm
- moved C1 18.0 mm to (155.2, 104.4), turned to 90 degrees
- moved C2 14.9 mm to (171.3, 102.5)
- moved C3 10.4 mm to (171.6, 107.3)
- moved U1 9.26 mm to (162.9, 108.1)
- moved Y1 9.22 mm to (164.9, 97.6), turned to 180 degrees
- moved R3 8.98 mm to (169.0, 99.8), turned to 270 degrees
- moved C5 7.99 mm to (166.1, 100.0), turned to 0 degrees
- moved C6 7.79 mm to (165.9, 115.6)
- moved R1 6.47 mm to (172.2, 109.3)
- moved C4 6.12 mm to (164.0, 100.0), turned to 0 degrees
- moved C7 5.79 mm to (173.8, 108.0)
- moved R2 5.51 mm to (172.2, 110.5)
Routing:
- net r1: track 156.2 -> 129.2 mm, vias 4 -> 2
- net c4: track 84.8 -> 70.6 mm
- net reset: track 26.5 -> 39.5 mm
- net r0: track 172.1 -> 160.7 mm, vias 2 -> 0
- net c3: track 156.3 -> 164.6 mm
- net MOSI: track 193.0 -> 199.6 mm
- net c5: track 88.1 -> 94.5 mm, vias 2 -> 4
- net Net-(C5-Pad1): track 6.89 -> 13.1 mm, vias 0 -> 2
- net MISO: track 169.7 -> 175.6 mm
- net GND: track 59.1 -> 64.9 mm, vias 4 -> 6
- net VCC: track 234.0 -> 238.5 mm, vias 15 -> 12
- net serial: track 75.0 -> 79.1 mm
- net d+: track 129.6 -> 133.4 mm
- net d-: track 127.3 -> 130.1 mm
- net Net-(C4-Pad1): track 6.79 -> 4.27 mm
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