File: pinkytyl_v2.sch (KiCad schematic (older format))
At the start: 62 parts, among them J1 50-00174, J2 Conn_01x02, J3 USB_B_Mini, J5 Conn_02x05_Odd_Even, K0 KEYSW, K10 KEYSW, K11 KEYSW, K12 KEYSW, K13 KEYSW, K14 KEYSW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

Commit message: Adds JLCPCB part numbers
Parts:
- C1, C2, C3, C6: LSCS Part # (none) -> C1525
- C4, C5: LSCS Part # (none) -> C1555
- C7: LSCS Part # (none) -> C52923
- D0, D10, D11, D12, D13, D14, D15, D20, D21, D22, D23, D24, D25, D30, D31, D32, D33, D34, D35, D40, D41: LSCS Part # (none) -> C81598
- R1, R2: LSCS Part # (none) -> C25092
- R3: LSCS Part # (none) -> C25744
- U1: LSCS Part # (none) -> C112161
- Y1: LSCS Part # (none) -> C13738
Changed lines of the file:
@@
 F 2 "Capacitor_SMD:C_0402_1005Metric" H 1750 1400 50  0001 C CNN
 F 3 "~" H 1750 1400 50  0001 C CNN
+F 4 "C1555" H 1750 1400 50  0001 C CNN "LSCS Part #"
 	1    1750 1400
 	0    1    1    0
@@
 F 2 "Capacitor_SMD:C_0402_1005Metric" H 1750 1600 50  0001 C CNN
 F 3 "~" H 1750 1600 50  0001 C CNN
+F 4 "C1555" H 1750 1600 50  0001 C CNN "LSCS Part #"
 	1    1750 1600
 	0    1    1    0
@@
 F 2 "Capacitor_SMD:C_0402_1005Metric" H 2200 1800 50  0001 C CNN
 F 3 "~" H 2200 1800 50  0001 C CNN
+F 4 "C1525" H 2200 1800 50  0001 C CNN "LSCS Part #"
 	1    2200 1800
 	0    1    1    0
@@
 F 2 "Capacitor_SMD:C_0402_1005Metric" H 2200 2500 50  0001 C CNN
 F 3 "~" H 2200 2500 50  0001 C CNN
+F 4 "C52923" H 2200 2500 50  0001 C CNN "LSCS Part #"
 	1    2200 2500
 	0    1    1    0
@@
 F 2 "Capacitor_SMD:C_0402_1005Metric" H 950 1100 50  0001 C CNN
 F 3 "~" H 950 1100 50  0001 C CNN
+F 4 "C1525" H 950 1100 50  0001 C CNN "LSCS Part #"
 	1    950  1100
 	1    0    0    -1
@@
 F 2 "Capacitor_SMD:C_0402_1005Metric" H 550 1100 50  0001 C CNN
 F 3 "~" H 550 1100 50  0001 C CNN
+F 4 "C1525" H 550 1100 50  0001 C CNN "LSCS Part #"
 	1    550  1100
 	1    0    0    -1
@@
 F 2 "Resistor_SMD:R_0402_1005Metric" H 2050 2200 50  0001 C CNN
 F 3 "~" H 2050 2200 50  0001 C CNN
+F 4 "C25092" H 2050 2200 50  0001 C CNN "LSCS Part #"
 	1    2050 2200
 	0    1    1    0
@@
 F 2 "Resistor_SMD:R_0402_1005Metric" H 2050 2300 50  0001 C CNN
 F 3 "~" H 2050 2300 50  0001 C CNN
+F 4 "C25092" H 2050 2300 50  0001 C CNN "LSCS Part #"
 	1    2050 2300
 	0    1    1    0
@@
 F 2 "Diode_SMD:D_SOD-123" H 10300 3750 50  0001 C CNN
 F 3 "~" H 10300 3750 50  0001 C CNN
+F 4 "C81598" H 10300 3750 50  0001 C CNN "LSCS Part #"
 	1    10300 3750
 	0    1    1    0
@@
 F 2 "Diode_SMD:D_SOD-123" H 9350 3750 50  0001 C CNN
 F 3 "~" H 9350 3750 50  0001 C CNN
+F 4 "C81598" H 9350 3750 50  0001 C CNN "LSCS Part #"
 	1    9350 3750
 	0    1    1    0
@@
 F 2 "Diode_SMD:D_SOD-123" H 8500 3750 50  0001 C CNN
 F 3 "~" H 8500 3750 50  0001 C CNN
+F 4 "C81598" H 8500 3750 50  0001 C CNN "LSCS Part #"
 	1    8500 3750
 	0    1    1    0
@@
 F 2 "Diode_SMD:D_SOD-123" H 7650 3750 50  0001 C CNN
 F 3 "~" H 7650 3750 50  0001 C CNN
+F 4 "C81598" H 7650 3750 50  0001 C CNN "LSCS Part #"
 	1    7650 3750
 	0    1    1    0
@@
 F 2 "Diode_SMD:D_SOD-123" H 6750 3750 50  0001 C CNN
 F 3 "~" H 6750 3750 50  0001 C CNN
+F 4 "C81598" H 6750 3750 50  0001 C CNN "LSCS Part #"
 	1    6750 3750
 	0    1    1    0
@@
 F 2 "Diode_SMD:D_SOD-123" H 5850 3750 50  0001 C CNN
 F 3 "~" H 5850 3750 50  0001 C CNN
+F 4 "C81598" H 5850 3750 50  0001 C CNN "LSCS Part #"
 	1    5850 3750
 	0    1    1    0
@@
 F 2 "Diode_SMD:D_SOD-123" H 10300 4500 50  0001 C CNN
 F 3 "~" H 10300 4500 50  0001 C CNN
+F 4 "C81598" H 10300 4500 50  0001 C CNN "LSCS Part #"
 	1    10300 4500
 	0    1    1    0
@@
 F 2 "Diode_SMD:D_SOD-123" H 9350 4500 50  0001 C CNN
 F 3 "~" H 9350 4500 50  0001 C CNN
+F 4 "C81598" H 9350 4500 50  0001 C CNN "LSCS Part #"
 	1    9350 4500
 	0    1    1    0
@@
 F 2 "Diode_SMD:D_SOD-123" H 8500 4500 50  0001 C CNN
 F 3 "~" H 8500 4500 50  0001 C CNN
+F 4 "C81598" H 8500 4500 50  0001 C CNN "LSCS Part #"
 	1    8500 4500
 	0    1    1    0
@@
 F 2 "Diode_SMD:D_SOD-123" H 7650 4500 50  0001 C CNN
 F 3 "~" H 7650 4500 50  0001 C CNN
+F 4 "C81598" H 7650 4500 50  0001 C CNN "LSCS Part #"
 	1    7650 4500
 	0    1    1    0
@@
 F 2 "Diode_SMD:D_SOD-123" H 6750 4500 50  0001 C CNN
 F 3 "~" H 6750 4500 50  0001 C CNN
+F 4 "C81598" H 6750 4500 50  0001 C CNN "LSCS Part #"
 	1    6750 4500
 	0    1    1    0
@@
 F 2 "Diode_SMD:D_SOD-123" H 5850 4500 50  0001 C CNN
 F 3 "~" H 5850 4500 50  0001 C CNN
+F 4 "C81598" H 5850 4500 50  0001 C CNN "LSCS Part #"
 	1    5850 4500
 	0    1    1    0
@@
 F 2 "Diode_SMD:D_SOD-123" H 10300 5300 50  0001 C CNN
 F 3 "~" H 10300 5300 50  0001 C CNN
+F 4 "C81598" H 10300 5300 50  0001 C CNN "LSCS Part #"
 	1    10300 5300
 	0    1    1    0
@@
 F 2 "Diode_SMD:D_SOD-123" H 9350 5300 50  0001 C CNN
 F 3 "~" H 9350 5300 50  0001 C CNN
+F 4 "C81598" H 9350 5300 50  0001 C CNN "LSCS Part #"
 	1    9350 5300
 	0    1    1    0
@@
 F 2 "Diode_SMD:D_SOD-123" H 8500 5300 50  0001 C CNN
 F 3 "~" H 8500 5300 50  0001 C CNN
+F 4 "C81598" H 8500 5300 50  0001 C CNN "LSCS Part #"
 	1    8500 5300
 	0    1    1    0
@@
 F 2 "Diode_SMD:D_SOD-123" H 7650 5300 50  0001 C CNN
 F 3 "~" H 7650 5300 50  0001 C CNN
+F 4 "C81598" H 7650 5300 50  0001 C CNN "LSCS Part #"
 	1    7650 5300
 	0    1    1    0
@@
 F 2 "Diode_SMD:D_SOD-123" H 5850 5600 50  0001 C CNN
 F 3 "~" H 5850 5600 50  0001 C CNN
+F 4 "C81598" H 5850 5600 50  0001 C CNN "LSCS Part #"
 	1    5850 5600
 	0    -1   -1   0
@@
 F 2 "Diode_SMD:D_SOD-123" H 10300 6000 50  0001 C CNN
 F 3 "~" H 10300 6000 50  0001 C CNN
+F 4 "C81598" H 10300 6000 50  0001 C CNN "LSCS Part #"
 	1    10300 6000
 	0    1    1    0
@@
 F 2 "Diode_SMD:D_SOD-123" H 9350 6000 50  0001 C CNN
 F 3 "~" H 9350 6000 50  0001 C CNN
+F 4 "C81598" H 9350 6000 50  0001 C CNN "LSCS Part #"
 	1    9350 6000
 	0    1    1    0
@@
 F 2 "Diode_SMD:D_SOD-123" H 6750 3100 50  0001 C CNN
 F 3 "~" H 6750 3100 50  0001 C CNN
+F 4 "C81598" H 6750 3100 50  0001 C CNN "LSCS Part #"
 	1    6750 3100
 	0    1    1    0
@@
 F 2 "Diode_SMD:D_SOD-123" H 6750 5600 50  0001 C CNN
 F 3 "~" H 6750 5600 50  0001 C CNN
+F 4 "C81598" H 6750 5600 50  0001 C CNN "LSCS Part #"
 	1    6750 5600
 	0    -1   -1   0
@@
 F 2 "Capacitor_SMD:C_0402_1005Metric" H 1250 1100 50  0001 C CNN
 F 3 "~" H 1250 1100 50  0001 C CNN
+F 4 "C1525" H 1250 1100 50  0001 C CNN "LSCS Part #"
 	1    1250 1100
 	1    0    0    -1
@@
 F 2 "Resistor_SMD:R_0402_1005Metric" H 2200 850 50  0001 C CNN
 F 3 "~" H 2200 850 50  0001 C CNN
+F 4 "C25744" H 2200 850 50  0001 C CNN "LSCS Part #"
 	1    2200 850
 	-1   0    0    1
@@
 F 2 "Package_DFN_QFN:QFN-44-1EP_7x7mm_P0.5mm_EP5.2x5.2mm" H 2900 2700 50  0001 C CIN
 F 3 "http://ww1.microchip.com/downloads/en/DeviceDoc/Atmel-7766-8-bit-AVR-ATmega16U4-32U4_Datasheet.pdf" H 2900 2700 50  0001 C CNN
+F 4 "C112161" H 2900 2700 50  0001 C CNN "LSCS Part #"
 	1    2900 2700
 	1    0    0    -1
@@
 F 2 "Crystal:Crystal_SMD_3225-4Pin_3.2x2.5mm" H 2000 1500 50  0001 C CNN
 F 3 "~" H 2000 1500 50  0001 C CNN
+F 4 "C13738" H 2000 1500 50  0001 C CNN "LSCS Part #"
 	1    2000 1500
 	0    -1   -1   0

Commit message: Rough layout, might be ready for order
Parts:
- removed U1: ATmega32U4-MU, Package_DFN_QFN:QFN-44-1EP_7x7mm_P0.5mm_EP5.2x5.2mm, symbol MCU_Microchip_ATmega:ATmega32U4-MU
- added U?: ATmega32U4-AU, Package_QFP:TQFP-44_10x10mm_P0.8mm, symbol MCU_Microchip_ATmega:ATmega32U4-AU
Connections:
- net GND: now also U?.15 (GND), U?.23 (GND), U?.35 (GND), U?.43 (GND), U?.5 (UGND)
- net MISO: now also U?.11 (PB3)
- net MOSI: now also U?.10 (PB2)
- net VCC: now also U?.14 (VCC), U?.2 (UVCC), U?.24 (AVCC), U?.34 (VCC), U?.44 (AVCC), U?.7 (VBUS)
- net c0: now also U?.30 (PB6)
- net c3: now also U?.9 (PB1)
- net c4: now also U?.36 (PF7)
- net c5: now also U?.37 (PF6)
- net r0: now also U?.27 (PD7)
- net r1: now also U?.1 (PE6)
- net r2: now also U?.28 (PB4)
- net r3: now also U?.29 (PB5)
- net reset: now also U?.13 (~RESET)
- net serial: now also U?.18 (PD0)
- net at C4.1, Y1.3: now also U?.17 (XTAL1)
- net at C5.1, Y1.1: now also U?.16 (XTAL2)
- net at C6.1: now also U?.42 (AREF)
- net at C7.1: now also U?.6 (UCAP)
- net at R2.1: now also U?.3 (D-)
- net at R1.1: now also U?.4 (D+)
Changed lines of the file:
@@
-$EndComp
-$Comp
-L MCU_Microchip_ATmega:ATmega32U4-MU U1
-U 1 1 614A5BC3
-P 2900 2700
-F 0 "U1" H 2900 811 50  0000 C CNN
-F 1 "ATmega32U4-MU" H 2900 720 50  0000 C CNN
-F 2 "Package_DFN_QFN:QFN-44-1EP_7x7mm_P0.5mm_EP5.2x5.2mm" H 2900 2700 50  0001 C CIN
-F 3 "http://ww1.microchip.com/downloads/en/DeviceDoc/Atmel-7766-8-bit-AVR-ATmega16U4-32U4_Datasheet.pdf" H 2900 2700 50  0001 C CNN
-F 4 "C112161" H 2900 2700 50  0001 C CNN "LSCS Part #"
-	1    2900 2700
-	1    0    0    -1
 $EndComp
 $Comp
@@
 $EndComp
 Connection ~ 8750 2300
+$Comp
+L MCU_Microchip_ATmega:ATmega32U4-AU U?
+U 1 1 6151FE4B
+P 2900 2700
+F 0 "U?" H 2900 811 50  0000 C CNN
+F 1 "ATmega32U4-AU" H 2900 720 50  0000 C CNN
+F 2 "Package_QFP:TQFP-44_10x10mm_P0.8mm" H 2900 2700 50  0001 C CIN
+F 3 "http://ww1.microchip.com/downloads/en/DeviceDoc/Atmel-7766-8-bit-AVR-ATmega16U4-32U4_Datasheet.pdf" H 2900 2700 50  0001 C CNN
+	1    2900 2700
+	1    0    0    -1
+$EndComp
 $EndSCHEMATC

Commit message: Inc
Parts:
- C1, C2, C3, C6: LCSC (none) -> C1525; LSCS Part # C1525 -> (none)
- C4, C5: LCSC (none) -> C1555; LSCS Part # C1555 -> (none)
- C7: LCSC (none) -> C52923; LSCS Part # C52923 -> (none)
- D0, D10, D11, D12, D13, D14, D15, D20, D21, D22, D23, D24, D25, D30, D31, D32, D33, D34, D35, D40, D41: LCSC (none) -> C81598; LSCS Part # C81598 -> (none)
- R1, R2: LCSC (none) -> C25092; LSCS Part # C25092 -> (none)
- R3: LCSC (none) -> C25744; LSCS Part # C25744 -> (none)
- Y1: LCSC (none) -> C13738; LSCS Part # C13738 -> (none)
- gave numbers to parts that had none: 1
Changed lines of the file:
@@
 F 2 "Capacitor_SMD:C_0402_1005Metric" H 1750 1400 50  0001 C CNN
 F 3 "~" H 1750 1400 50  0001 C CNN
-F 4 "C1555" H 1750 1400 50  0001 C CNN "LSCS Part #"
+F 4 "C1555" H 1750 1400 50  0001 C CNN "LCSC"
 	1    1750 1400
 	0    1    1    0
@@
 F 2 "Capacitor_SMD:C_0402_1005Metric" H 1750 1600 50  0001 C CNN
 F 3 "~" H 1750 1600 50  0001 C CNN
-F 4 "C1555" H 1750 1600 50  0001 C CNN "LSCS Part #"
+F 4 "C1555" H 1750 1600 50  0001 C CNN "LCSC"
 	1    1750 1600
 	0    1    1    0
@@
 F 2 "Capacitor_SMD:C_0402_1005Metric" H 2200 1800 50  0001 C CNN
 F 3 "~" H 2200 1800 50  0001 C CNN
-F 4 "C1525" H 2200 1800 50  0001 C CNN "LSCS Part #"
+F 4 "C1525" H 2200 1800 50  0001 C CNN "LCSC"
 	1    2200 1800
 	0    1    1    0
@@
 F 2 "Capacitor_SMD:C_0402_1005Metric" H 2200 2500 50  0001 C CNN
 F 3 "~" H 2200 2500 50  0001 C CNN
-F 4 "C52923" H 2200 2500 50  0001 C CNN "LSCS Part #"
+F 4 "C52923" H 2200 2500 50  0001 C CNN "LCSC"
 	1    2200 2500
 	0    1    1    0
@@
 F 2 "Capacitor_SMD:C_0402_1005Metric" H 950 1100 50  0001 C CNN
 F 3 "~" H 950 1100 50  0001 C CNN
-F 4 "C1525" H 950 1100 50  0001 C CNN "LSCS Part #"
+F 4 "C1525" H 950 1100 50  0001 C CNN "LCSC"
 	1    950  1100
 	1    0    0    -1
@@
 F 2 "Capacitor_SMD:C_0402_1005Metric" H 550 1100 50  0001 C CNN
 F 3 "~" H 550 1100 50  0001 C CNN
-F 4 "C1525" H 550 1100 50  0001 C CNN "LSCS Part #"
+F 4 "C1525" H 550 1100 50  0001 C CNN "LCSC"
 	1    550  1100
 	1    0    0    -1
@@
 F 2 "Resistor_SMD:R_0402_1005Metric" H 2050 2200 50  0001 C CNN
 F 3 "~" H 2050 2200 50  0001 C CNN
-F 4 "C25092" H 2050 2200 50  0001 C CNN "LSCS Part #"
+F 4 "C25092" H 2050 2200 50  0001 C CNN "LCSC"
 	1    2050 2200
 	0    1    1    0
@@
 F 2 "Resistor_SMD:R_0402_1005Metric" H 2050 2300 50  0001 C CNN
 F 3 "~" H 2050 2300 50  0001 C CNN
-F 4 "C25092" H 2050 2300 50  0001 C CNN "LSCS Part #"
+F 4 "C25092" H 2050 2300 50  0001 C CNN "LCSC"
 	1    2050 2300
 	0    1    1    0
@@
 F 2 "Diode_SMD:D_SOD-123" H 10300 3750 50  0001 C CNN
 F 3 "~" H 10300 3750 50  0001 C CNN
-F 4 "C81598" H 10300 3750 50  0001 C CNN "LSCS Part #"
+F 4 "C81598" H 10300 3750 50  0001 C CNN "LCSC"
 	1    10300 3750
 	0    1    1    0
@@
 F 2 "Diode_SMD:D_SOD-123" H 9350 3750 50  0001 C CNN
 F 3 "~" H 9350 3750 50  0001 C CNN
-F 4 "C81598" H 9350 3750 50  0001 C CNN "LSCS Part #"
+F 4 "C81598" H 9350 3750 50  0001 C CNN "LCSC"
 	1    9350 3750
 	0    1    1    0
@@
 F 2 "Diode_SMD:D_SOD-123" H 8500 3750 50  0001 C CNN
 F 3 "~" H 8500 3750 50  0001 C CNN
-F 4 "C81598" H 8500 3750 50  0001 C CNN "LSCS Part #"
+F 4 "C81598" H 8500 3750 50  0001 C CNN "LCSC"
 	1    8500 3750
 	0    1    1    0
@@
 F 2 "Diode_SMD:D_SOD-123" H 7650 3750 50  0001 C CNN
 F 3 "~" H 7650 3750 50  0001 C CNN
-F 4 "C81598" H 7650 3750 50  0001 C CNN "LSCS Part #"
+F 4 "C81598" H 7650 3750 50  0001 C CNN "LCSC"
 	1    7650 3750
 	0    1    1    0
@@
 F 2 "Diode_SMD:D_SOD-123" H 6750 3750 50  0001 C CNN
 F 3 "~" H 6750 3750 50  0001 C CNN
-F 4 "C81598" H 6750 3750 50  0001 C CNN "LSCS Part #"
+F 4 "C81598" H 6750 3750 50  0001 C CNN "LCSC"
 	1    6750 3750
 	0    1    1    0
@@
 F 2 "Diode_SMD:D_SOD-123" H 5850 3750 50  0001 C CNN
 F 3 "~" H 5850 3750 50  0001 C CNN
-F 4 "C81598" H 5850 3750 50  0001 C CNN "LSCS Part #"
+F 4 "C81598" H 5850 3750 50  0001 C CNN "LCSC"
 	1    5850 3750
 	0    1    1    0
@@
 F 2 "Diode_SMD:D_SOD-123" H 10300 4500 50  0001 C CNN
 F 3 "~" H 10300 4500 50  0001 C CNN
-F 4 "C81598" H 10300 4500 50  0001 C CNN "LSCS Part #"
+F 4 "C81598" H 10300 4500 50  0001 C CNN "LCSC"
 	1    10300 4500
 	0    1    1    0
@@
 F 2 "Diode_SMD:D_SOD-123" H 9350 4500 50  0001 C CNN
 F 3 "~" H 9350 4500 50  0001 C CNN
-F 4 "C81598" H 9350 4500 50  0001 C CNN "LSCS Part #"
+F 4 "C81598" H 9350 4500 50  0001 C CNN "LCSC"
 	1    9350 4500
 	0    1    1    0
@@
 F 2 "Diode_SMD:D_SOD-123" H 8500 4500 50  0001 C CNN
 F 3 "~" H 8500 4500 50  0001 C CNN
-F 4 "C81598" H 8500 4500 50  0001 C CNN "LSCS Part #"
+F 4 "C81598" H 8500 4500 50  0001 C CNN "LCSC"
 	1    8500 4500
 	0    1    1    0
@@
 F 2 "Diode_SMD:D_SOD-123" H 7650 4500 50  0001 C CNN
 F 3 "~" H 7650 4500 50  0001 C CNN
-F 4 "C81598" H 7650 4500 50  0001 C CNN "LSCS Part #"
+F 4 "C81598" H 7650 4500 50  0001 C CNN "LCSC"
 	1    7650 4500
 	0    1    1    0
@@
 F 2 "Diode_SMD:D_SOD-123" H 6750 4500 50  0001 C CNN
 F 3 "~" H 6750 4500 50  0001 C CNN
-F 4 "C81598" H 6750 4500 50  0001 C CNN "LSCS Part #"
+F 4 "C81598" H 6750 4500 50  0001 C CNN "LCSC"
 	1    6750 4500
 	0    1    1    0
@@
 F 2 "Diode_SMD:D_SOD-123" H 5850 4500 50  0001 C CNN
 F 3 "~" H 5850 4500 50  0001 C CNN
-F 4 "C81598" H 5850 4500 50  0001 C CNN "LSCS Part #"
+F 4 "C81598" H 5850 4500 50  0001 C CNN "LCSC"
 	1    5850 4500
 	0    1    1    0
@@
 F 2 "Diode_SMD:D_SOD-123" H 10300 5300 50  0001 C CNN
 F 3 "~" H 10300 5300 50  0001 C CNN
-F 4 "C81598" H 10300 5300 50  0001 C CNN "LSCS Part #"
+F 4 "C81598" H 10300 5300 50  0001 C CNN "LCSC"
 	1    10300 5300
 	0    1    1    0
@@
 F 2 "Diode_SMD:D_SOD-123" H 9350 5300 50  0001 C CNN
 F 3 "~" H 9350 5300 50  0001 C CNN
-F 4 "C81598" H 9350 5300 50  0001 C CNN "LSCS Part #"
+F 4 "C81598" H 9350 5300 50  0001 C CNN "LCSC"
 	1    9350 5300
 	0    1    1    0
@@
 F 2 "Diode_SMD:D_SOD-123" H 8500 5300 50  0001 C CNN
 F 3 "~" H 8500 5300 50  0001 C CNN
-F 4 "C81598" H 8500 5300 50  0001 C CNN "LSCS Part #"
+F 4 "C81598" H 8500 5300 50  0001 C CNN "LCSC"
 	1    8500 5300
 	0    1    1    0
@@
 F 2 "Diode_SMD:D_SOD-123" H 7650 5300 50  0001 C CNN
 F 3 "~" H 7650 5300 50  0001 C CNN
-F 4 "C81598" H 7650 5300 50  0001 C CNN "LSCS Part #"
+F 4 "C81598" H 7650 5300 50  0001 C CNN "LCSC"
 	1    7650 5300
 	0    1    1    0
@@
 F 2 "Diode_SMD:D_SOD-123" H 5850 5600 50  0001 C CNN
 F 3 "~" H 5850 5600 50  0001 C CNN
-F 4 "C81598" H 5850 5600 50  0001 C CNN "LSCS Part #"
+F 4 "C81598" H 5850 5600 50  0001 C CNN "LCSC"
 	1    5850 5600
 	0    -1   -1   0
@@
 F 2 "Diode_SMD:D_SOD-123" H 10300 6000 50  0001 C CNN
 F 3 "~" H 10300 6000 50  0001 C CNN
-F 4 "C81598" H 10300 6000 50  0001 C CNN "LSCS Part #"
+F 4 "C81598" H 10300 6000 50  0001 C CNN "LCSC"
 	1    10300 6000
 	0    1    1    0
@@
 F 2 "Diode_SMD:D_SOD-123" H 9350 6000 50  0001 C CNN
 F 3 "~" H 9350 6000 50  0001 C CNN
-F 4 "C81598" H 9350 6000 50  0001 C CNN "LSCS Part #"
+F 4 "C81598" H 9350 6000 50  0001 C CNN "LCSC"
 	1    9350 6000
 	0    1    1    0
@@
 F 2 "Diode_SMD:D_SOD-123" H 6750 3100 50  0001 C CNN
 F 3 "~" H 6750 3100 50  0001 C CNN
-F 4 "C81598" H 6750 3100 50  0001 C CNN "LSCS Part #"
+F 4 "C81598" H 6750 3100 50  0001 C CNN "LCSC"
 	1    6750 3100
 	0    1    1    0
@@
 F 2 "Diode_SMD:D_SOD-123" H 6750 5600 50  0001 C CNN
 F 3 "~" H 6750 5600 50  0001 C CNN
-F 4 "C81598" H 6750 5600 50  0001 C CNN "LSCS Part #"
+F 4 "C81598" H 6750 5600 50  0001 C CNN "LCSC"
 	1    6750 5600
 	0    -1   -1   0
@@
 F 2 "Capacitor_SMD:C_0402_1005Metric" H 1250 1100 50  0001 C CNN
 F 3 "~" H 1250 1100 50  0001 C CNN
-F 4 "C1525" H 1250 1100 50  0001 C CNN "LSCS Part #"
+F 4 "C1525" H 1250 1100 50  0001 C CNN "LCSC"
 	1    1250 1100
 	1    0    0    -1
@@
 F 2 "Resistor_SMD:R_0402_1005Metric" H 2200 850 50  0001 C CNN
 F 3 "~" H 2200 850 50  0001 C CNN
-F 4 "C25744" H 2200 850 50  0001 C CNN "LSCS Part #"
+F 4 "C25744" H 2200 850 50  0001 C CNN "LCSC"
 	1    2200 850
 	-1   0    0    1
@@
 F 2 "Crystal:Crystal_SMD_3225-4Pin_3.2x2.5mm" H 2000 1500 50  0001 C CNN
 F 3 "~" H 2000 1500 50  0001 C CNN
-F 4 "C13738" H 2000 1500 50  0001 C CNN "LSCS Part #"
+F 4 "C13738" H 2000 1500 50  0001 C CNN "LCSC"
 	1    2000 1500
 	0    -1   -1   0
@@
 Connection ~ 8750 2300
 $Comp
-L MCU_Microchip_ATmega:ATmega32U4-AU U?
+L MCU_Microchip_ATmega:ATmega32U4-AU U1
 U 1 1 6151FE4B
 P 2900 2700
-F 0 "U?" H 2900 811 50  0000 C CNN
+F 0 "U1" H 2900 811 50  0000 C CNN
 F 1 "ATmega32U4-AU" H 2900 720 50  0000 C CNN
 F 2 "Package_QFP:TQFP-44_10x10mm_P0.8mm" H 2900 2700 50  0001 C CIN
